Commit message: Add gripper_tip frame, live pose plot + MeshCat sim, teach/playback tooling

File: urdf/reBot-DevArm_fixend_description/urdf/reBot-DevArm_fixend.urdf (robot description, URDF)
Before this commit: robot reBot-DevArm_fixend, 8 links, 7 joints
Links:
- added link gripper_tip, mass 0.000001
Joints:
- added joint gripper_tip_joint: type fixed, parent end_link, child gripper_tip, origin xyz=0.07 0 0 rpy=0 0 0, axis 0 0 0
